Commit message: Verify no-mass warnings dont produce zero-mass links; refresh robot/ re-import

File: robot/robot.urdf (robot description, URDF)
Before this commit: robot onshape_export, 15 links, 14 joints
Links:
- link hip_roll_assembly: mass 0.01148 -> 0.0964752; geometry collision mesh filename=package://assets/l_roll_motor_bottom.stl; collision mesh filename=package://assets/l_roll_motor_top.stl
- link hip_roll_assembly_2: mass 0.01148 -> 0.0964752; geometry collision mesh filename=package://assets/l_roll_motor_bottom.stl; collision mesh filename=package://assets/l_roll_motor_top.stl
- link knee_and_ankle_assembly: mass 0.01825 -> 0.103245; geometry collision mesh filename=package://assets/left_knee_to_ankle_left_sheet.stl; collision mesh filename=package://assets/left_knee_to_ankle_left_sheet.stl
- link knee_and_ankle_assembly_2: mass 0.01825 -> 0.103245; geometry collision mesh filename=package://assets/left_knee_to_ankle_left_sheet.stl; collision mesh filename=package://assets/left_knee_to_ankle_left_sheet.stl
- link knee_and_ankle_assembly_3: mass 0.01825 -> 0.103245; geometry collision mesh filename=package://assets/left_knee_to_ankle_left_sheet.stl; collision mesh filename=package://assets/left_knee_to_ankle_left_sheet.stl
- link knee_and_ankle_assembly_4: mass 0.01825 -> 0.103245; geometry collision mesh filename=package://assets/left_knee_to_ankle_left_sheet.stl; collision mesh filename=package://assets/left_knee_to_ankle_left_sheet.stl
- link left_roll_to_pitch_assembly: mass 0.02016 -> 0.105155; geometry collision mesh filename=package://assets/left_roll_to_pitch.stl; collision mesh filename=package://assets/part_10.stl
- link neck_pitch_assembly: mass 0.01118 -> 0.0961752; geometry collision mesh filename=package://assets/neck_left_sheet.stl; collision mesh filename=package://assets/neck_right_sheet.stl
- link neck_yaw_assembly: mass 0.0389231 -> 0.123918; geometry collision mesh filename=package://assets/head_yaw_to_roll.stl; collision mesh filename=package://assets/part_10.stl
- link right_roll_to_pitch_assembly: mass 0.0366271 -> 0.121622; geometry collision mesh filename=package://assets/part_10.stl; collision mesh filename=package://assets/part_11.stl
- link trunk_assembly: mass 0.141168 -> 0.525868; geometry collision mesh filename=package://assets/bno055.stl; collision mesh filename=package://assets/part_1.stl
- link xm430_어셈: mass 0.07109 -> 0.232708; geometry collision mesh filename=package://assets/head_bot_sheet.stl; collision mesh filename=package://assets/part_10.stl
Joints:
- joint head_yaw: origin xyz=0.0410829 -0.0410829 -0.019 rpy=1.5708 -0 0.785398 -> xyz=0.0410829 -0.0410829 -0.019 rpy=1.5708 0 0.785398
- joint neck_pitch: origin xyz=0.0009 0.019 0.0911524 rpy=1.5708 -0.785398 -0 -> xyz=0.0009 0.019 0.0911524 rpy=1.5708 -0.785398 0

Commit message: Close out board-inclusion investigation: was a stale name, not a bug

File: robot/robot.urdf (robot description, URDF)
Before this commit: robot robot, 15 links, 14 joints
Joints:
- joint head_pitch: limit lower=-1.5708 upper=-0 effort=10 velocity=10 -> lower=-1.5708 upper=0 effort=10 velocity=10

Commit message: Confirm Korean-name USD path warning resolved after OnShape rename

File: robot/robot.urdf (robot description, URDF)
Before this commit: robot robot, 15 links, 14 joints
Links:
- removed link xm430_어셈
- added link xm430_assem, mass 0.232708; collision mesh filename=package://assets/head_bot_sheet.stl; collision mesh filename=package://assets/part_10.stl
Joints:
- joint head_pitch: limit lower=-1.5708 upper=0 effort=10 velocity=10 -> lower=-1.5708 upper=-0 effort=10 velocity=10
- joint head_roll: child xm430_어셈 -> xm430_assem
- joint right_knee: origin xyz=0 0.07865 0.038 rpy=3.14159 0 -1.5708 -> xyz=0 0.07865 0.038 rpy=3.14159 -0 -1.5708
