Commit message: robot: re-import the finished CAD — 2.7140 kg, and a clean import log
The mass is real now: densities replace the old overrides, so mass and
inertia come from the same source. Every link's radius of gyration lands
between 0.42 and 0.56 of its mesh radius, tightly clustered — the
signature of consistent density, and the thing that goes wrong when only
mass is overridden. Total is 2.7140 kg against the CAD's 2.7152 (+1.2 g).

Getting here took three imports, and the first two each found something:

  * config.json pointed at a stale *workspace* of the same document. Same
    document and element id, different w/ — so the URL looked unchanged
    while the geometry was months old. Fixed to w/1a1b1904...

  * left and right roll_to_pitch differed by 14.27 g with byte-identical
    mesh volume (29.02 cm3 each) and the same 17-part list. Only density
    can do that; the right side was the wrong one.

  * "Multiple base links" came from a single JST-B3B-EH-A connector
    instance with no mate. Booleans in the Part Studio cannot fix this —
    onshape-to-robot builds its tree from *assembly mates*, so an unmated
    instance becomes its own base link and gets dropped. It was the only
    part missing from the URDF (0 references, STL present).

Now: ERROR 0, no-mass 0, multiple-base 0, Traceback 0. The 4 remaining
warnings are the harmless same-name STL renames.

Unchanged and verified rather than assumed: the 14 joint names still match
ACTUATOR_JOINT_NAMES, joint limits still match hardware_map exactly, the
trunk frame is still +x forward / +y left / +z up, and the leg chain moved
at most 0.20 mm (hip-to-foot 246.47 -> 246.52) — so the placo reference
motion stays valid and does not need regenerating.

Two things did need fixing:

  * imu_map.MOUNT_POS — the IMU moved 1.76 mm (z 91.44 -> 89.64). The
    axis map is still identity since rpy is still 0. Added the one-liner
    that reads the value out of the URDF, because this needs redoing on
    every import.

  * inject_materials.py matched on the mesh's direct parent, which now
    holds an intermediate node_STL_BINARY_ level, so it coloured 0 of 642
    prims. It walks ancestors until it finds a known stem: 574/642, the
    same ratio as before.

Leg-trunk clearance on the new geometry, 5 mm standard, across all six
commands: 0.0% violation, 0.0% contact, 5.8 mm minimum, 14.0 mm median.

Co-Authored-By: Claude Opus 5 <noreply@anthropic.com>
Claude-Session: https://claude.ai/code/session_01Ktvp75ksqEpSsRvABxjE7i

File: robot/robot.urdf (robot description, URDF)
Before this commit: robot robot, 20 links, 19 joints
Links:
- link foot_assembly: mass 0.07524 -> 0.0694995; geometry collision mesh filename=package://assets/foot_bottom_pla.stl; collision mesh filename=package://assets/foot_bottom_tpu.stl
- link foot_assembly_2: mass 0.07524 -> 0.0694995; geometry collision mesh filename=package://assets/foot_bottom_pla.stl; collision mesh filename=package://assets/foot_bottom_tpu.stl
- link head_pitch_assembly: mass 0.0190918 -> 0.0139999
- link hip_roll_assembly: mass 0.0964752 -> 0.100996; geometry collision mesh filename=package://assets/l_roll_motor_bottom.stl; collision mesh filename=package://assets/l_roll_motor_top.stl
- link hip_roll_assembly_2: mass 0.0964752 -> 0.100996; geometry collision mesh filename=package://assets/l_roll_motor_bottom.stl; collision mesh filename=package://assets/l_roll_motor_top.stl
- link knee_and_ankle_assembly: mass 0.103245 -> 0.102496; geometry collision mesh filename=package://assets/left_knee_to_ankle_left_sheet.stl; collision mesh filename=package://assets/left_knee_to_ankle_left_sheet.stl
- link knee_and_ankle_assembly_2: mass 0.103245 -> 0.102496; geometry collision mesh filename=package://assets/left_knee_to_ankle_left_sheet.stl; collision mesh filename=package://assets/left_knee_to_ankle_left_sheet.stl
- link knee_and_ankle_assembly_3: mass 0.103245 -> 0.102496; geometry collision mesh filename=package://assets/left_knee_to_ankle_left_sheet.stl; collision mesh filename=package://assets/left_knee_to_ankle_left_sheet.stl
- link knee_and_ankle_assembly_4: mass 0.103245 -> 0.102496; geometry collision mesh filename=package://assets/left_knee_to_ankle_left_sheet.stl; collision mesh filename=package://assets/left_knee_to_ankle_left_sheet.stl
- link left_roll_to_pitch_assembly: mass 0.121995 -> 0.106996; geometry collision mesh filename=package://assets/left_roll_to_pitch.stl; collision mesh filename=package://assets/part_10.stl
- link neck_pitch_assembly: mass 0.0961752 -> 0.0949947; geometry collision mesh filename=package://assets/neck_left_sheet.stl; collision mesh filename=package://assets/neck_right_sheet.stl
- link neck_yaw_assembly: mass 0.123918 -> 0.124002; geometry collision mesh filename=package://assets/head_yaw_to_roll.stl; collision mesh filename=package://assets/part_10.stl
- link right_roll_to_pitch_assembly: mass 0.121622 -> 0.106996; geometry collision mesh filename=package://assets/part_10.stl; collision mesh filename=package://assets/part_11.stl
- link trunk_assembly: mass 0.866868 -> 1.13596; geometry collision mesh filename=package://assets/batt.stl; collision mesh filename=package://assets/bno055.stl
- link xm430_assem: mass 0.232708 -> 0.380052; geometry collision mesh filename=package://assets/head_bot_sheet.stl; collision mesh filename=package://assets/part_10.stl
Joints:
- joint head_frame: origin xyz=0.05369 -0 0.0227159 rpy=1e-12 1.5708 0 -> xyz=0.05369 -0 0.0228062 rpy=1e-12 1.5708 0
- joint head_roll: origin xyz=0.04095 -0 -0.0203 rpy=0 -1.5708 0 -> xyz=0.04095 0 -0.0205 rpy=-0 -1.5708 0
- joint imu_frame: origin xyz=-0.03883 -0 0.0914424 rpy=-0 0 0 -> xyz=-0.038493 0 0.0896424 rpy=-0 -0 0
- joint left_foot_frame: origin xyz=0.0005 0.036225 -0.01955 rpy=1.5708 -0 -0 -> xyz=0.0005 0.036225 -0.01955 rpy=1.5708 0 0
- joint left_hip_pitch: origin xyz=0.0753 -1.7e-11 -0.035685 rpy=3.14159 -1.5708 0 -> xyz=0.0755 -1.7e-11 -0.035685 rpy=3.14159 -1.5708 0
- joint left_knee: origin xyz=0 0.07865 1.537e-09 rpy=0 0 -0 -> xyz=-0 0.07865 1.537e-09 rpy=0 0 -0
- joint neck_pitch: origin xyz=0.0009 0.019 0.0911524 rpy=1.5708 -0 -0 -> xyz=0.0009 0.019 0.0911524 rpy=1.5708 -0 0
- joint right_hip_pitch: origin xyz=-0.0753 0 0.035685 rpy=0 1.5708 0 -> xyz=-0.0751 -0.0002 0.035685 rpy=0 1.5708 0
- joint right_hip_roll: origin xyz=0.019 -0.00011 0.04599 rpy=1.5708 0 -1.5708 -> xyz=0.019 -0.00011 0.04599 rpy=1.5708 -0 -1.5708
- joint right_hip_yaw: origin xyz=-0.019 -0.035 0.0474424 rpy=3.14159 0 0 -> xyz=-0.019 -0.035 0.0474424 rpy=3.14159 -0 0

Commit message: v33n: train the new robot on ref_g115, and put the status on the README
v33n is v33 with only the robot and the gait swapped. v33 itself stopped at
iter 663, but its curves were healthy — no warnings, +24.8% over the last
500 iters, ahead of v32 at the same point on both reward and episode
length. The Z-neck pose was never the problem. It just cannot be resumed:
the robot gained 16% mass and the IMU moved 41 mm, which changes the
observation, so anything trained before 815cead no longer matches the
config.

  reference   ref_h175 (planned for the 2.3388 kg robot) -> ref_g115
  robot       2.3388 -> 2.7140 kg
  READY       measured, not guessed: settle 138.3 mm from a 200 mm drop,
              sigma 1.6, spawn set from the max rather than the mean
  head_pitch  45 deg with room, see below
  everything else — hip-inward penalty, locked head, network, gamma — as v32/v33

head_pitch's URDF limit was exactly 45 deg, which is also the pose the
Z-neck wants, so v33 sat on the stop with 0.4 mrad to spare and the PD
leaned on it every step. The user confirmed the mechanism actually travels
about +-60 deg and the 45 was a CAD clamp; the limit is now +-50, giving
the pose 5 deg. Note this has to be re-applied after any `odm import` until
the mate limit is fixed in OnShape, and that the USD must be reconverted —
Isaac Lab validates default joint positions against the USD, not the URDF,
and refuses to build the env otherwise.

viz_ref_pkl.py plays a reference straight from its pkl, so it works while
training holds the only Isaac Sim slot. It also made something visible that
is worth knowing: the reference's legs deliver about half the commanded
travel — 40.3 mm per cycle against the 81.0 mm that 0.15 m/s implies — so
the feet visibly slide in a contact-free kinematic replay. The policy makes
up the difference through tracking_lin_vel.

The README now opens with a status block, so someone landing on the repo
can see what is running, what is done, what the current wall is (the servo
bus at 10.8 Hz against the 50 Hz the policy needs), and what comes next.

Co-Authored-By: Claude Opus 5 <noreply@anthropic.com>
Claude-Session: https://claude.ai/code/session_01Ktvp75ksqEpSsRvABxjE7i

File: robot/robot.urdf (robot description, URDF)
Before this commit: robot robot, 20 links, 19 joints
Joints:
- joint head_pitch: limit lower=-0.785398 upper=0.785398 effort=10 velocity=10 -> lower=-0.872665 upper=0.872665 effort=10 velocity=10
