Commit message: Fix Stage 2 pipeline: pin placo==0.6.3, patch URDF with Placo frame aliases

File: reference_motion_generator/open_duck_reference_motion_generator/robots/open_duck_mini_v2/open_duck_mini_v2.urdf (robot description, URDF)
Before this commit: robot robot, 15 links, 14 joints
Links:
- added link head, mass 1e-9
- added link left_foot, mass 1e-9
- added link right_foot, mass 1e-9
- added link trunk, mass 1e-9
Joints:
- added joint head_frame: type fixed, parent head_pitch_assembly, child head, origin xyz=0.04245 0 0.03595 rpy=0 1.570796326794896558 0, axis 0 0 0
- added joint left_foot_frame: type fixed, parent foot_assembly, child left_foot, origin xyz=0.0005 -0.036225 0.01955 rpy=-1.570796326794896558 0 0, axis 0 0 0
- added joint right_foot_frame: type fixed, parent foot_assembly_2, child right_foot, origin xyz=0.0005 -0.036225 0.01955 rpy=-1.570796326794896558 0 0, axis 0 0 0
- added joint trunk_frame: type fixed, parent trunk_assembly, child trunk, origin xyz=-0.024 0 0.08819 rpy=0 0 0, axis 0 0 0

Commit message: fix: medium.json walk_com_height 0.16 + feet_spacing 0.18

File: reference_motion_generator/open_duck_reference_motion_generator/robots/open_duck_mini_v2/open_duck_mini_v2.urdf (robot description, URDF)
Before this commit: robot robot, 19 links, 18 joints
Links:
- added link imu, mass 1e-9
- link left_roll_to_pitch_assembly: mass 0.105155 -> 0.121995
- link trunk_assembly: mass 0.666868 -> 0.866868; geometry collision mesh filename=package://assets/batt.stl; collision mesh filename=package://assets/bno055.stl
Joints:
- added joint imu_frame: type fixed, parent trunk_assembly, child imu, origin xyz=-0.03883 -0 0.0914424 rpy=-0 0 0, axis 0 0 0
- joint head_frame: origin xyz=0.04245 0 0.03595 rpy=0 1.570796326794896558 0 -> xyz=0.05369 -0 0.0227159 rpy=1e-12 1.5708 0; parent head_pitch_assembly -> xm430_assem
- joint head_pitch: limit lower=-1.5708 upper=0 effort=10 velocity=10 -> lower=-0.785398 upper=0.785398 effort=10 velocity=10
- joint head_yaw: origin xyz=0.0410829 -0.0410829 -0.019 rpy=1.5708 0 0.785398 -> xyz=0 -0.0581 -0.019 rpy=1.5708 -0 0
- joint left_ankle: limit lower=-2.29509 upper=0.846508 effort=10 velocity=10 -> lower=-1.5708 upper=1.5708 effort=10 velocity=10; origin xyz=0.07865 1.74719e-06 1.537e-09 rpy=-0 0 -1.57077 -> xyz=-0 0.07865 1.537e-09 rpy=-0 0 0
- joint left_foot_frame: origin xyz=0.0005 -0.036225 0.01955 rpy=-1.570796326794896558 0 0 -> xyz=0.0005 0.036225 -0.01955 rpy=1.5708 -0 0
- joint left_hip_pitch: limit lower=-1.37008 upper=0.375245 effort=10 velocity=10 -> lower=-0.523599 upper=1.22173 effort=10 velocity=10
- joint left_knee: limit lower=-2.22148e-05 upper=3.14157 effort=10 velocity=10 -> lower=-1.5708 upper=1.5708 effort=10 velocity=10; origin xyz=-0.0589054 0.052115 1.537e-09 rpy=-0 -0 0.846485 -> xyz=0 0.07865 1.537e-09 rpy=0 0 -1e-12
- joint neck_pitch: limit lower=-1.13446 upper=0.349066 effort=10 velocity=10 -> lower=-0.349066 upper=1.13446 effort=10 velocity=10; origin xyz=0.0009 0.019 0.0911524 rpy=1.5708 -0.785398 0 -> xyz=0.0009 0.019 0.0911524 rpy=1.5708 -0 0
- joint right_ankle: limit lower=-0.846508 upper=2.29509 effort=10 velocity=10 -> lower=-1.5708 upper=1.5708 effort=10 velocity=10; origin xyz=0 -0.07865 -1.537e-09 rpy=-0 0 -0.724289 -> xyz=0 -0.07865 -1.537e-09 rpy=-0 -0 -0
- joint right_foot_frame: origin xyz=0.0005 -0.036225 0.01955 rpy=-1.570796326794896558 0 0 -> xyz=0.0005 -0.036225 0.01955 rpy=-1.5708 -0 -0
- joint right_hip_pitch: limit lower=-1.37008 upper=0.375245 effort=10 velocity=10 -> lower=-0.523599 upper=1.22173 effort=10 velocity=10; origin xyz=-0.0753 -0 0.035685 rpy=1.5708 0.724311 1.5708 -> xyz=-0.0753 0 0.035685 rpy=0 1.5708 0
- joint right_knee: limit lower=-3.14157 upper=2.22148e-05 effort=10 velocity=10 -> lower=-1.5708 upper=1.5708 effort=10 velocity=10; origin xyz=0 0.07865 0.038 rpy=3.14159 -0 -1.57077 -> xyz=0 0.07865 0.038 rpy=-3.14159 -0 -0
- joint trunk_frame: origin xyz=-0.024 0 0.08819 rpy=0 0 0 -> xyz=-0.024 -0 0.0893424 rpy=-0 -0 -0

Commit message: fix: 무릎 ±120° + URDF-따라가는 방향강제, 무릎 ROM 부활 pkl

File: reference_motion_generator/open_duck_reference_motion_generator/robots/open_duck_mini_v2/open_duck_mini_v2.urdf (robot description, URDF)
Before this commit: robot robot, 20 links, 19 joints
Joints:
- joint left_ankle: origin xyz=-0 0.07865 1.537e-09 rpy=-0 0 0 -> xyz=0 0.07865 1.537e-09 rpy=-0 0 0
- joint left_foot_frame: origin xyz=0.0005 0.036225 -0.01955 rpy=1.5708 -0 0 -> xyz=0.0005 0.036225 -0.01955 rpy=1.5708 -0 -0
- joint left_knee: limit lower=-1.5708 upper=1.5708 effort=10 velocity=10 -> lower=-2.0944 upper=2.0944 effort=10 velocity=10; origin xyz=0 0.07865 1.537e-09 rpy=0 0 -1e-12 -> xyz=0 0.07865 1.537e-09 rpy=0 0 -0
- joint neck_pitch: origin xyz=0.0009 0.019 0.0911524 rpy=1.5708 -0 0 -> xyz=0.0009 0.019 0.0911524 rpy=1.5708 -0 -0
- joint right_ankle: origin xyz=0 -0.07865 -1.537e-09 rpy=-0 -0 -0 -> xyz=0 -0.07865 -1.537e-09 rpy=-0 0 -0
- joint right_knee: limit lower=-1.5708 upper=1.5708 effort=10 velocity=10 -> lower=-2.0944 upper=2.0944 effort=10 velocity=10

File: robot/robot.urdf (robot description, URDF)
Before this commit: robot robot, 15 links, 14 joints
Links:
- added link head, mass 1e-9
- added link imu, mass 1e-9
- added link left_foot, mass 1e-9
- added link right_foot, mass 1e-9
- added link trunk, mass 1e-9
- link left_roll_to_pitch_assembly: mass 0.105155 -> 0.121995
- link trunk_assembly: mass 0.525868 -> 0.866868; geometry collision mesh filename=package://assets/batt.stl; collision mesh filename=package://assets/bno055.stl
Joints:
- added joint head_frame: type fixed, parent xm430_assem, child head, origin xyz=0.05369 -0 0.0227159 rpy=1e-12 1.5708 0, axis 0 0 0
- added joint imu_frame: type fixed, parent trunk_assembly, child imu, origin xyz=-0.03883 -0 0.0914424 rpy=-0 0 0, axis 0 0 0
- added joint left_foot_frame: type fixed, parent foot_assembly, child left_foot, origin xyz=0.0005 0.036225 -0.01955 rpy=1.5708 -0 -0, axis 0 0 0
- added joint right_foot_frame: type fixed, parent foot_assembly_2, child right_foot, origin xyz=0.0005 -0.036225 0.01955 rpy=-1.5708 -0 -0, axis 0 0 0
- added joint trunk_frame: type fixed, parent trunk_assembly, child trunk, origin xyz=-0.024 -0 0.0893424 rpy=-0 -0 -0, axis 0 0 0
- joint head_pitch: limit lower=-1.5708 upper=-0 effort=10 velocity=10 -> lower=-0.785398 upper=0.785398 effort=10 velocity=10
- joint head_yaw: origin xyz=0.0410829 -0.0410829 -0.019 rpy=1.5708 0 0.785398 -> xyz=0 -0.0581 -0.019 rpy=1.5708 -0 0
- joint left_ankle: limit lower=-1.91986 upper=1.22173 effort=10 velocity=10 -> lower=-1.5708 upper=1.5708 effort=10 velocity=10; origin xyz=0.07865 0 1.537e-09 rpy=-0 0 -1.5708 -> xyz=0 0.07865 1.537e-09 rpy=-0 0 0
- joint left_hip_pitch: limit lower=-1.74533 upper=6e-12 effort=10 velocity=10 -> lower=-0.523599 upper=1.22173 effort=10 velocity=10
- joint left_knee: limit lower=-1e-12 upper=3.14159 effort=10 velocity=10 -> lower=-2.0944 upper=2.0944 effort=10 velocity=10; origin xyz=-0.0739068 0.0268999 1.537e-09 rpy=0 0 1.22173 -> xyz=0 0.07865 1.537e-09 rpy=0 0 -0
- joint neck_pitch: limit lower=-1.13446 upper=0.349066 effort=10 velocity=10 -> lower=-0.349066 upper=1.13446 effort=10 velocity=10; origin xyz=0.0009 0.019 0.0911524 rpy=1.5708 -0.785398 0 -> xyz=0.0009 0.019 0.0911524 rpy=1.5708 -0 -0
- joint right_ankle: limit lower=-1.22173 upper=1.91986 effort=10 velocity=10 -> lower=-1.5708 upper=1.5708 effort=10 velocity=10; origin xyz=0 -0.07865 -1.537e-09 rpy=0 0 -0.349066 -> xyz=0 -0.07865 -1.537e-09 rpy=-0 0 -0
- joint right_hip_pitch: limit lower=-1.74533 upper=6e-12 effort=10 velocity=10 -> lower=-0.523599 upper=1.22173 effort=10 velocity=10; origin xyz=-0.0753 -0 0.035685 rpy=1.5708 0.349066 1.5708 -> xyz=-0.0753 0 0.035685 rpy=0 1.5708 0
- joint right_hip_roll: origin xyz=0.019 -0.00011 0.04599 rpy=1.5708 1e-12 -1.5708 -> xyz=0.019 -0.00011 0.04599 rpy=1.5708 0 -1.5708
- joint right_knee: limit lower=-3.14159 upper=1e-12 effort=10 velocity=10 -> lower=-2.0944 upper=2.0944 effort=10 velocity=10; origin xyz=0 0.07865 0.038 rpy=3.14159 -0 -1.5708 -> xyz=0 0.07865 0.038 rpy=-3.14159 -0 -0
