Commit message: CAD 질량 갱신(2.7430 kg) + 정지 시 몸통 수직 리워드(v35) + ONNX 익스포터
body tail 실측 113 g 을 OnShape 밀도(1352.7 -> 1820.6 kg/m^3)로 반영하고
재임포트했다. 로봇 총질량 2.7140 -> 2.7430 kg, 전체 CoM 이 뒤로 1.06 mm.
USD 를 백업본과 대조해 그 외에는 아무것도 안 바뀌었음을 확인했다.

임포트가 로컬 수정을 덮어쓰는 문제를 고쳤다. head_pitch 한계 ±50도가 CAD 의
±45도로 되돌아갔는데, 시뮬은 URDF 가 아니라 USD 에서 한계를 읽으므로 재변환
전에는 티도 안 난다. apply_local_urdf_overrides.py 에 표로 모아 파이프라인에
묶었다(멱등). patch_urdf_for_placo.py 도 임포트에 안 묶여 있어서 추가했다 —
이 SSD 는 exFAT 라 심볼릭 링크가 안 돼 실제 복사가 필요하다.

v35 = v34c10 + 정지 시 몸통 수직. v34u 는 같은 목표를 정지 목표 관절각으로
우회해서 풀었다가 몸통 피치가 +8.19 -> +20.93 도로 나빠졌다. 관절각은 간접
손잡이라서다. 이번엔 projected_gravity 의 x,y 를 직접 벌한다. 기본 계수는 0
이라 기존 태스크의 리워드는 한 항도 안 바뀐다.

레퍼런스 생성을 이 PC 에서도 되게 했다(scripts/setup/gen_reference_local.sh,
odm refgen). "placo 를 못 깐다" 던 진단이 틀렸다 — ~/.odm-tools 의 numpy 가
2.x 라 cmeel 스택이 소스 빌드로 떨어진 것이었고, numpy==1.26.4 를 박은 전용
venv 에는 42개가 전부 wheel 로 들어온다. 랩PC 와 같은 프리셋·URDF 로 생성해
500x55 프레임이 비트 단위로 일치함을 확인했다. 원격판도 그대로 남겨 뒀다.

레퍼런스 격자 수정이 랩PC 파일에만 있고 레포엔 없던 것도 고쳤다
(auto_gait.json yaw ±0.3 -> ±0.28, 0 을 포함하는 대칭 격자).

ONNX 익스포터를 추가했다(scripts/hw/export_onnx.py). IsaacLab 의 play.py 가
자동으로 만들어 주던 건데 이 레포는 odm play 를 쓰므로 v28 이후 하나도 없었다.
Isaac Sim 없이 CPU 로만 돌아 학습과 병행된다. 체크포인트의 obs_normalizer 를
그래프 안에 넣어 실기는 원시 관측만 넣으면 된다 — torch 대비 상대오차 2.5e-07.

실기 배포 계약은 docs/handoff/onnx_deploy_2026-08-08.md 에 정리했다.

Co-Authored-By: Claude Opus 5 <noreply@anthropic.com>
Claude-Session: https://claude.ai/code/session_01Ktvp75ksqEpSsRvABxjE7i

File: reference_motion_generator/open_duck_reference_motion_generator/robots/open_duck_mini_v2/open_duck_mini_v2.urdf (robot description, URDF)
Before this commit: robot robot, 20 links, 19 joints
Links:
- link trunk_assembly: mass 1.13596 -> 1.165
Joints:
- joint head_pitch: limit lower=-0.785398 upper=0.785398 effort=10 velocity=10 -> lower=-0.872665 upper=0.872665 effort=10 velocity=10

File: robot/robot.urdf (robot description, URDF)
Before this commit: robot robot, 20 links, 19 joints
Links:
- link trunk_assembly: mass 1.13596 -> 1.165
